File: CodeName02.kicad_pcb (KiCad board)
At the start: 4 copper layers, 60 x 80 mm, 129 parts, among them J1 Power & ESC Signal, J2 I2C Connection, J3 STM32 Debug Connection, J4 Buzzer Connection, J5 GPS Connection, J6 UART Connection, J7 SPI Connection, J8 Jumper Pin Select, Q1 MMBT3904, Q2 AO3011A, Q3 AO3011A, SW1 TACTILE SWITCH, SW2 TACTILE SWITCH, SW3 TACTILE SWITCH, SW4 TACTILE SWITCH, U1 ICM-42605, U10 MX74610T, U11 CH224K, U12 ESP32-C3FH4, U13 TLV75733PDBVR, U2 STM32H743VITx, U3 XT25F128FWOIGT-W, U4 BMP388, U5 SP1117, U6 MX74610T, U7 INA226AIDGSR, U8 SY8368AQQC, U9 TP3USB30M10, X1 XVFEELNANF-8MHZ, X2 X322540MPB4SI

Commit message: feat: finalize
Parts:
- added C61: 10nF, Capacitor_SMD:C_0603_1608Metric, F.Cu at (136.3, 128.1)
- added C62: 10nF, Capacitor_SMD:C_0603_1608Metric, F.Cu at (138.7, 128.9)
- added C63: 100nF, Capacitor_SMD:C_0603_1608Metric, F.Cu at (131.8, 120.4)
- added C64: 470nF, Capacitor_SMD:C_0603_1608Metric, F.Cu at (129.4, 122.8)
- added C65: 100nF, Capacitor_SMD:C_0603_1608Metric, F.Cu at (126.1, 126.2)
- added C66: 10nF, Capacitor_SMD:C_0603_1608Metric, F.Cu at (131.8, 122.0)
- added C67: 47pF, Capacitor_SMD:C_0402_1005Metric, F.Cu at (129.0, 126.0)
- added C68: 10nF, Capacitor_SMD:C_0603_1608Metric, F.Cu at (127.7, 126.2)
- added FL1: 2450FM07D0034T, easyeda2kicad:FILTER-SMD_4P-L1.0-W0.5-L, F.Cu at (132.8, 134.7)
- added G***: LOGO, Library:Chevron-Top, F.Cu at (142.8, 92.7)
- added G***: LOGO, Library:signature, F.Cu at (151.1, 85.8)
- added G***: LOGO, Library:ghidorah, F.Cu at (148.8, 80.2)
- added G***: LOGO, Library:ghidorah-txt, F.Cu at (148.8, 84.7)
- added J10: AUX Timer Connection, easyeda2kicad:PinHeader_3Row_Custom, F.Cu at (144.9, 132.1)
- added J9: Conn_Coaxial_Small, Connector_Coaxial:U.FL_Hirose_U.FL-R-SMT-1_Vertical, F.Cu at (132.8, 137.7)
- added REF**: ESD-Logo_8.9x8mm_SilkScreen, Symbol:ESD-Logo_8.9x8mm_SilkScreen, F.Cu at (149.0, 124.3)
- added TP1: TestPoint VBAT_RAW, TestPoint:TestPoint_Pad_D2.0mm, F.Cu at (150.1, 74.1)
- added TP2: TestPoint SYS_POWER, TestPoint:TestPoint_Pad_D2.0mm, F.Cu at (169.8, 77.9)
- added TP3: TestPoint 5V, TestPoint:TestPoint_Pad_D2.0mm, F.Cu at (176.8, 88.0)
- added TP4: TestPoint 3.3V, TestPoint:TestPoint_Pad_D2.0mm, F.Cu at (135.4, 75.8)
- added U14: SX1280IMLTRT, easyeda2kicad:QFN-24_L4.0-W4.0-P0.50-BL-EP2.6, F.Cu at (132.5, 125.8)
- added X3: XC21M4-52.000-F10NNHPL, easyeda2kicad:CRYSTAL-SMD_4P-L2.0-W1.6-BL, F.Cu at (137.1, 124.0)
- J2: footprint Connector_JST:JST_GH_SM04B-GHS-TB_1x04-1MP_P1.25mm_Horizontal -> Connector_JST:JST_GH_BM04B-GHS-TBT_1x04-1MP_P1.25mm_Vertical
- L2: footprint LED_SMD:LED_0402_1005Metric -> Inductor_SMD:L_0402_1005Metric
- U3: value XT25F128FWOIGT-W -> W25Q128JVPIQTR
- moved R22 256.2 mm to (125.4, 113.0), turned to 90 degrees
- moved R23 254.6 mm to (128.0, 117.6)
- moved U12 252.2 mm to (129.8, 109.8), turned to -90 degrees
- moved X2 248.4 mm to (137.7, 103.4), turned to -90 degrees
- moved R21 246.3 mm to (125.0, 108.0)
- moved C58 246.2 mm to (132.1, 114.9), turned to 90 degrees
- moved C52 245.4 mm to (128.9, 114.9), turned to -90 degrees
- moved C51 245.0 mm to (130.5, 114.9), turned to -90 degrees
- moved C54 244.9 mm to (127.3, 114.9), turned to -90 degrees
- moved SW4 244.6 mm to (134.3, 95.3), turned to 180 degrees
- moved SW3 244.5 mm to (134.3, 90.3), turned to 180 degrees
- moved R25 243.6 mm to (135.1, 111.1), turned to -90 degrees
- moved FB3 243.3 mm to (134.4, 115.7), turned to 180 degrees
- moved D3 243.1 mm to (128.0, 119.3)
- moved C57 243.0 mm to (136.8, 114.9), turned to 90 degrees
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Connections:
- net STM32_SDMMC1_CK renamed STM32_SDMMC1_CLK
- J1 pad MP: (no net) -> GND
- J4 pad MP: (no net) -> GND
- J5 pad MP: (no net) -> GND
- J6 pad MP: (no net) -> GND
- J7 pad MP: (no net) -> GND
- U12 pad 13: SX_DIO0 -> SX_BUSY
- U2 pad 47: unconnected-(U2-PB11-Pad47) -> STM32_INA_ALERT
- U2 pad 53: unconnected-(U2-PB14-Pad53) -> STM32_ISP2_MISO
Routing:
- net GND: track 1.60 -> 203.6 mm, vias 1 -> 226
- net STM32_I2C1_SCL: track 0.00 -> 110.2 mm, vias 0 -> 8
- net STM32_I2C1_SDA: track 0.00 -> 108.7 mm, vias 0 -> 4
- net +3.3V: track 0.00 -> 88.3 mm, vias 0 -> 23
- net +5V: track 0.00 -> 69.1 mm, vias 0 -> 8
- net STM32_SWDIO: track 0.00 -> 67.3 mm, vias 0 -> 4
- net STM32_BARO_INT: track 0.00 -> 62.3 mm, vias 0 -> 4
- net STM32_SWCLK: track 0.00 -> 60.4 mm, vias 0 -> 4
- net STM32_USB_DP: track 0.00 -> 60.3 mm, vias 0 -> 2
- net STM32_TIM1_CH4: track 0.00 -> 59.2 mm, vias 0 -> 2
- net STM32_TIM1_CH1: track 0.00 -> 58.7 mm, vias 0 -> 2
- net STM32_TIM1_CH2: track 0.00 -> 58.2 mm, vias 0 -> 2
- net STM32_TIM1_CH3: track 0.00 -> 58.1 mm, vias 0 -> 2
- net STM32_USB_DN: track 0.00 -> 49.9 mm, vias 0 -> 2
- net STM32_NRST: track 0.00 -> 47.4 mm, vias 0 -> 2
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- added copper zone on B.Cu, net +5V
- added copper zone on F.Cu, net +SYS_POWER
- added copper zone on B.Cu, net GND
- added copper zone on F.Cu, net GND
- added copper zone on F.Cu, net RF_VDD
Other:
- board text added: "BUZZER"
- board text added: "CLK"
- board text added: "DIO"
- board text added: "EBOOT"
- board text added: "ERST"
- board text added: "ESP"
- board text added: "GND"
- board text added: "GPS"
- board text added: "I2C"
- board text added: "POWER"
- board text added: "SBOOT"
- board text added: "SPI"
- board text added: "SRST"
- board text added: "STM"
- board text added: "UART"
