File: CodeName02.kicad_sch (KiCad schematic)
At the start: 5 parts, among them U1 STM32H743VITx, U2 SX1280IMLTRT, U3 ESP32-C3FH4, U4 SY8368AQQC

Commit message: feat: schematic update
Parts:
- removed U2: SX1280IMLTRT, easyeda2kicad:QFN-24_L4.0-W4.0-P0.50-BL-EP2.6, symbol easyeda2kicad:SX1280IMLTRT
- removed U3: ESP32-C3FH4, easyeda2kicad:QFN-32_L5.0-W5.0-P0.50-TL-EP3.7, symbol easyeda2kicad:ESP32-C3FH4
- added C1, C14, C23, C25, C26, C27, C29, C30, C32, C34, C35, C37, C38, C41, C43, C44, C46, C47, C48, C5, C50, C52, C7, C8, C9: 100nF, Capacitor_SMD:C_0603_1608Metric, symbol Device:C_Small
- added C10, C45: 2.2uF, Capacitor_SMD:C_0603_1608Metric, symbol Device:C_Small
- added C11, C12: 22uF, Capacitor_SMD:C_0805_2012Metric, symbol Device:C_Small
- added C13, C24, C28, C31, C33, C36, C39, C40, C49, C57, C58: 4.7uF, Capacitor_SMD:C_0603_1608Metric, symbol Device:C_Small
- added C15, C19, C20: 10uF, Capacitor_SMD:C_0805_2012Metric, symbol Device:C_Small
- added C16, C18, C21, C22: 22pF, Capacitor_SMD:C_0603_1608Metric, symbol Device:C_Small
- added C17: 1uF, Capacitor_SMD:C_0603_1608Metric, symbol Device:C_Small
- added C2, C3, C4: 100uF, Capacitor_SMD:C_1206_3216Metric, symbol Device:C_Small
- added C42, C51: 10nF, Capacitor_SMD:C_0603_1608Metric, symbol Device:C_Small
- added C53, C54: 10uF, Capacitor_SMD:C_0603_1608Metric, symbol Device:C_Small
- added C55, C56: 22uF, Capacitor_SMD:C_0603_1608Metric, symbol Device:C_Small
- added C6: 200pF, Capacitor_SMD:C_0603_1608Metric, symbol Device:C_Small
- added D1, D2: XL-1608PGC-06, easyeda2kicad:LED0603-RD_GREEN, symbol easyeda2kicad:XL-1608PGC-06
- added D3: DSK34, easyeda2kicad:SOD-123FL_L2.7-W1.8-LS3.8-RD, symbol easyeda2kicad:DSK34_C727076
- added FB1, FB2, FB3: FerriteBead, Inductor_SMD:L_0603_1608Metric, symbol Device:FerriteBead_Small
- added J1: Jumper Pin Select, easyeda2kicad:PinHeader_1x03_P2.54mm_Vertical_Custom, symbol Connector:Conn_01x03_Pin
- added J2: UART Connection, Connector_JST:JST_GH_SM04B-GHS-TB_1x04-1MP_P1.25mm_Horizontal, symbol Connector:Conn_01x04_Pin
- added J3: STM32 Debug Connection, easyeda2kicad:PinHeader_1x03_P2.54mm_Vertical_Custom, symbol Connector:Conn_01x03_Pin
- added J4: GPS Connection, Connector_JST:JST_GH_SM06B-GHS-TB_1x06-1MP_P1.25mm_Horizontal, symbol Connector:Conn_01x06_Pin
- added J5: Power & ESC Signal, Connector_JST:JST_GH_SM06B-GHS-TB_1x06-1MP_P1.25mm_Horizontal, symbol Connector:Conn_01x06_Pin
- added J6: SPI Connection, Connector_JST:JST_GH_SM06B-GHS-TB_1x06-1MP_P1.25mm_Horizontal, symbol Connector:Conn_01x06_Pin
- added J7: Buzzer Connection, Connector_JST:JST_GH_SM02B-GHS-TB_1x02-1MP_P1.25mm_Horizontal, symbol Connector:Conn_01x02_Pin
- added J8: I2C Connection, Connector_JST:JST_GH_SM04B-GHS-TB_1x04-1MP_P1.25mm_Horizontal, symbol Connector:Conn_01x04_Pin
- added Q1, Q2: AO3011A, easyeda2kicad:SOT-23-3_L2.9-W1.6-P1.90-LS2.8-BR, symbol easyeda2kicad:AO3011A
- added Q3: MMBT3904, Package_TO_SOT_SMD:SOT-23, symbol Transistor_BJT:MMBT3904
- added R1: 100K, symbol Device:R_Small
- added R10, R11, R12, R13, R15, R16, R21, R25, R7, R9: 10K, Resistor_SMD:R_0603_1608Metric, symbol Device:R_Small
- added R14, R22: 100, Resistor_SMD:R_0603_1608Metric, symbol Device:R_Small
- added R17, R18, R19, R20: 22, Resistor_SMD:R_0603_1608Metric, symbol Device:R_Small
- added R2: LR2512D-0.5MR, easyeda2kicad:RES-SMD_L6.4-W3.2_C500733, symbol easyeda2kicad:LR2512D-3W-0.5MR-1%
- added R23, R24: 2.2K, Resistor_SMD:R_0603_1608Metric, symbol Device:R_Small
- added R3, R5: 10K, symbol Device:R_Small
- added R4: 1K, symbol Device:R_Small
- added R6: 12K, symbol Device:R_Small
- added R8: 1K, Resistor_SMD:R_0603_1608Metric, symbol Device:R_Small
- added SW1, SW2, SW3, SW4: TACTILE SWITCH, easyeda2kicad:KEY-SMD_L4.0-W3.0-LS4.9-1, symbol easyeda2kicad:HX3X4X2-2P-1.6NTACTILESWITCH
- added U1: TP3USB30M10, easyeda2kicad:MSOP-10_L3.0-W3.0-P0.50-LS4.9-BL, symbol easyeda2kicad:TP3USB30M10
- added U10: ICM-42605, easyeda2kicad:LGA-14_L3.0-W2.5-P0.50-TL, symbol easyeda2kicad:ICM-42605
- added U11: ESP32-C3FH4, easyeda2kicad:QFN-32_L5.0-W5.0-P0.50-TL-EP3.7, symbol easyeda2kicad:ESP32-C3FH4
- added U13: TLV75733PDBVR, easyeda2kicad:SOT-23-5_L2.9-W1.6-P0.95-LS2.8-BL, symbol easyeda2kicad:TLV75733PDBVR
- added U2: INA226AIDGSR, easyeda2kicad:MSOP-10_L3.0-W3.0-P0.50-LS5.0-BL, symbol easyeda2kicad:INA226AIDGSR
- added U4, U9: MX74610T, easyeda2kicad:SOT-23-6_L2.9-W1.6-P0.95-LS2.8-BL-1, symbol easyeda2kicad:MX74610T
- added U5: SP1117, Package_TO_SOT_SMD:SOT-223-3_TabPin2, symbol Regulator_Linear:AMS1117
- added U6: CH224K, Package_SO:SSOP-10-1EP_3.9x4.9mm_P1mm_EP2.1x3.3mm, symbol Interface_USB:CH224K
- added U7: XT25F128FWOIGT-W, easyeda2kicad:WSON-8_L6.0-W5.0-P1.27-BL-EP, symbol easyeda2kicad:XT25F128FWOIGT-W
- added U8: BMP388, easyeda2kicad:SENSORM-SMD_BMP388, symbol easyeda2kicad:BMP388
- added USB1: USB-TYPE-C-018, easyeda2kicad:USB-C_SMD-TYPE-C-31-M-12, symbol easyeda2kicad:USB-TYPE-C-018
- added X1: XVFEELNANF-8MHZ, easyeda2kicad:CRYSTAL-SMD_4P-L5.0-W3.2-BL-1, symbol easyeda2kicad:XVFEELNANF-8MHZ
- added X2: X322540MPB4SI, easyeda2kicad:OSC-SMD_4P-L3.2-W2.5-BL_SIT8008BI, symbol easyeda2kicad:X322540MPB4SI
- renumbered U1 to U12, U4 to U3
Connections:
- net at L1.1: now also U3.2 (LX), C1.1
- net +5V: now reaches L1.2
- net +5V: now also C19.1, C2.1, C3.1, C4.1, C5.1, C56.1, C6.2, FB3.2, J2.1 (Pin_1), J4.1 (Pin_1), J6.1 (Pin_1), J7.1 (Pin_1), J8.1 (Pin_1), R1.2, U13.3 (EN), U5.3 (VI)
- net GND: now reaches U3.1 (GND)
- net GND: now also U12.10 (VSS), U12.19 (VSSA), U12.26 (VSS), U12.49 (VSS), U12.74 (VSS), U12.99 (VSS), U3.3 (GND), C11.2, C12.2, C13.2, C14.1, C15.2, C16.2, C17.2, C18.1, C19.2, C2.2, C20.2, C21.2, C22.2, C23.1, C24.1, C25.2, C26.2, C27.2, C28.1, C29.2, C3.2, C30.2, C31.1, C32.2, C33.1, C34.2, C35.2, C36.1, C37.2, C38.2, C39.1, C4.2, C40.1, C41.2, C42.2, C43.2, C44.2, C46.2, C47.2, C48.2, C49.1, C5.2, C50.2, C51.2, C52.2, C53.2, C54.2, C55.2, C56.2, C57.2, C58.1, C7.2, C9.2, D1.1 (K), D2.1 (K), J1.3 (Pin_3), J2.2 (Pin_2), J3.3 (Pin_3), J4.2 (Pin_2), J5.2 (Pin_2), J6.2 (Pin_2), J8.2 (Pin_2), Q3.3 (C), R10.1, R21.1, R6.1, SW1.2, SW3.2, SW4.2, U1.5 (GND), U1.9 (OEB), U10.10 (RESV), U10.11 (RESV), U10.2 (RESV), U10.3 (RESV), U10.6 (GND), U10.7 (RESV), U10.9 (INT2/FSYNC), U11.33 (EP), U13.2 (GND), U2.1 (A1), U2.2 (A0), U2.7 (GND), U5.1 (ADJ), U6.11 (GND), U6.2 (CFG2), U6.3 (CFG3), U6.9 (CFG1), U7.4 (VSS), U7.9 (EP), U8.3 (VSS), U8.5 (SDO), U8.8 (VSS), U8.9 (VSS), USB1.0 (SH), USB1.1 (SH), USB1.2 (SH), USB1.3 (SH), USB1.A1 (GND), USB1.A12 (GND), USB1.B1 (GND), USB1.B12 (GND), X1.2 (GND), X1.4 (GND), X2.2 (GND), X2.4 (GND)
- net at U3.10 (ILMT): now also R5.1
- net at U3.12 (EN): now also R3.1
- net +SYS_POWER: now reaches U3.4 (IN)
- net +SYS_POWER: now also U3.5 (IN), U3.6 (IN), C11.1, C12.1, C8.2, Q2.3 (D), R2.2, R3.2, R5.2, U2.9 (VIN-), U9.1 (CATHODE)
- net at U3.7 (BS): now also C1.2
- net at U3.8 (VCC): now also C13.1
- net at U3.9 (FB): now also R1.1, R4.1, R6.2
- net STM32_QSPI_IO2: now reaches U12.1 (PE2)
- net STM32_QSPI_IO2: now also U7.3 (WP#(IO2))
- net +3.3V: now reaches U12.100 (VDD)
- net +3.3V: now also U12.11 (VDD), U12.20 (VREF+), U12.27 (VDD), U12.50 (VDD), U12.6 (VBAT), U12.75 (VDD), C20.1, C24.2, C25.1, C26.1, C27.1, C28.2, C29.1, C30.1, C31.2, C32.1, C33.2, C34.1, C35.1, C36.2, C37.1, C40.2, C41.1, C46.1, C7.1, C9.1, FB1.2, FB2.2, J1.1 (Pin_1), R11.1, R12.1, R13.1, R15.1, R23.1, R24.1, R7.1, R9.1, SW2.2, U1.10 (VCC), U10.5 (VDDIO), U2.6 (VS+), U5.2 (VO), U7.8 (VCC), U8.1 (VDDIO), U8.10 (VDD), U8.6 (CSB)
- net STM32_XTAL_IN: now reaches U12.12 (PH0)
- net STM32_XTAL_IN: now also C21.1, X1.1
- net STM32_XTAL_OUT: now reaches U12.13 (PH1)
- net STM32_XTAL_OUT: now also C16.1, X1.3
- net STM32_NRST: now reaches U12.14 (NRST)
- net STM32_NRST: now also C14.2, R9.2, SW1.1
- net at U12.21 (VDDA): now also C38.1, C39.2, FB1.1
- net STM32_TIM5_CH1: now reaches U12.22 (PA0)
- net STM32_TIM5_CH2: now reaches U12.23 (PA1)
- net STM32_TIM5_CH3: now reaches U12.24 (PA2)
- net STM32_TIM5_CH4: now reaches U12.25 (PA3)
- net STM32_IMU_CS: now reaches U12.28 (PA4)
- net STM32_IMU_CS: now also R15.2, U10.12 (AP_CS)
- net STM32_ISP1_SCK: now reaches U12.29 (PA5)
- net STM32_ISP1_SCK: now also U10.13 (AP_SCL/AP_SCLK)
- net STM32_ISP1_MISO: now reaches U12.30 (PA6)
- net STM32_ISP1_MISO: now also U10.1 (AP_SDO/AP_AD0)
- net STM32_ISP1_MOSI: now reaches U12.31 (PA7)
- net STM32_ISP1_MOSI: now also U10.14 (AP_SDA/AP_SDIO/AP_SDI)
- net STM32_QSPI_CLK: now reaches U12.36 (PB2)
- net STM32_QSPI_CLK: now also U7.6 (SCLK)
- net STM32_TIM1_CH1: now reaches U12.39 (PE9)
- net STM32_TIM1_CH1: now also J5.3 (Pin_3)
- net STM32_TIM1_CH2: now reaches U12.41 (PE11)
- net STM32_TIM1_CH3: now reaches U12.43 (PE13)
- net STM32_TIM1_CH3: now also J5.5 (Pin_5)
- net STM32_TIM1_CH4: now reaches U12.44 (PE14)
- net STM32_TIM1_CH4: now also J5.6 (Pin_6)
- net STM32_QSPI_NCS: now reaches U12.46 (PB10)
- net STM32_QSPI_NCS: now also R12.2, U7.1 (~{CS})
- net at U12.48 (VCAP): now also C57.1
- net STM32_ISP2_NSS: now reaches U12.51 (PB12)
- net STM32_ISP2_NSS: now also J6.3 (Pin_3)
- net STM32_ISP2_SCK: now reaches U12.52 (PB13)
- net STM32_ISP2_SCK: now also J6.4 (Pin_4)
- net STM32_ISP2_MOSI: now reaches U12.54 (PB15)
- net STM32_ISP2_MOSI: now also J6.6 (Pin_6)
- net STM32_USART3_TX: now reaches U12.55 (PD8)
- net STM32_USART3_TX: now also J2.3 (Pin_3)
- net STM32_USART3_RX: now reaches U12.56 (PD9)
- net STM32_USART3_RX: now also J2.4 (Pin_4)
- net STM32_BARO_INT: now reaches U12.57 (PD10)
- net STM32_BARO_INT: now also U8.7 (INT)
- net STM32_QSPI_IO0: now reaches U12.58 (PD11)
- net STM32_QSPI_IO0: now also U7.5 (SI(IO0))
- net STM32_QSPI_IO1: now reaches U12.59 (PD12)
- net STM32_QSPI_IO1: now also U7.2 (SO(IO1))
- net STM32_QSPI_IO3: now reaches U12.60 (PD13)
- net STM32_QSPI_IO3: now also U7.7 (HOLD#(IO3))
- net STM32_TIM4_CH1: now reaches U12.61 (PD14)
- net STM32_TIM4_CH2: now reaches U12.62 (PD15)
- net STM32_SDMMC1_D0: now reaches U12.65 (PC8)
- net STM32_SDMMC1_D1: now reaches U12.66 (PC9)
- net STM32_IMU_INT: now reaches U12.67 (PA8)
- net STM32_IMU_INT: now also U10.4 (INT1/INT)
- net STM32_USART1_TX: now reaches U12.68 (PA9)
- net STM32_USART1_TX: now also U11.27 (U0RXD)
- net STM32_USART1_RX: now reaches U12.69 (PA10)
- net STM32_USART1_RX: now also U11.28 (U0TXD)
- net STM32_LED: now reaches U12.7 (PC13)
- net STM32_LED: now also R14.1
- net at U12.70 (PA11): now also R17.2
- net at U12.71 (PA12): now also R19.2
- net STM32_SWDIO: now reaches U12.72 (PA13)
- net STM32_SWDIO: now also J3.1 (Pin_1)
- net at U12.73 (VCAP): now also C58.2
- net STM32_SWCLK: now reaches U12.76 (PA14)
- net STM32_SWCLK: now also J3.2 (Pin_2)
- net STM32_SDMMC1_D2: now reaches U12.78 (PC10)
- net STM32_SDMMC1_D3: now reaches U12.79 (PC11)
- net STM32_SDMMC1_CK: now reaches U12.80 (PC12)
- net STM32_SDMMC1_CMD: now reaches U12.83 (PD2)
- net STM32_USART2_TX: now reaches U12.86 (PD5)
- net STM32_USART2_TX: now also J4.3 (Pin_3)
- net STM32_USART2_RX: now reaches U12.87 (PD6)
- net STM32_USART2_RX: now also J4.4 (Pin_4)
- net STM32_BUZZER_CTRL: now reaches U12.88 (PD7)
- net STM32_BUZZER_CTRL: now also R25.2
- net STM32_BOOT: now reaches U12.94 (BOOT0)
- net STM32_BOOT: now also R10.2, SW2.1
- net STM32_I2C1_SCL: now reaches U12.95 (PB8)
- net STM32_I2C1_SCL: now also J4.5 (Pin_5), J8.3 (Pin_3), R23.2, U2.5 (SCL), U8.2 (SCK)
- net STM32_I2C1_SDA: now reaches U12.96 (PB9)
- net STM32_I2C1_SDA: now also J4.6 (Pin_6), J8.4 (Pin_4), R24.2, U2.4 (SDA), U8.4 (SDI)
- new net: Q3.1 (B), R25.1
- new net: D3.2 (A), Q3.2 (E)
- new net: R22.1, U11.16 (GPIO10)
- new net: D2.2 (A), R22.2
- new net: C6.1, R4.2
- new net: C49.2, C50.1, FB2.1, U10.8 (VDD)
- new net: C54.1, C55.1, FB3.1, U13.1 (IN)
- new net: Q2.1 (G), U9.2 (GATEPD), U9.3 (GATE)
- new net: D3.1 (K), J7.2 (Pin_2)
- new net: R20.2, U11.25 (GPIO18)
- new net: R18.2, U11.26 (GPIO19)
- new net: C17.1, R8.2, U6.1 (VDD)
- new net: Q1.1 (G), U4.2 (GATEPD), U4.3 (GATE)
- new net: C45.1, U9.6 (VCAPL)
- new net: C45.2, U9.5 (VCAPH)
- new net: C10.2, U4.5 (VCAPH)
- new net: C10.1, U4.6 (VCAPL)
- new net: D1.2 (A), R14.2
- new net +BATT_RAW: J5.1 (Pin_1), Q1.2 (S), U4.4 (ANODE)
- new net +BATT_SAFE: C8.1, Q1.3 (D), R2.1, U2.10 (VIN+), U2.8 (VBUS), U4.1 (CATHODE)
- new net +USB_VBUS: C15.1, Q2.2 (S), R8.1, U6.8 (VBUS), U9.4 (ANODE), USB1.A4 (VBUS), USB1.A9 (VBUS), USB1.B4 (VBUS), USB1.B9 (VBUS)
- new net ESP32_BOOT: R13.2, SW4.1, U11.15 (GPIO9)
- new net ESP32_EN: C23.2, R11.2, SW3.1, U11.7 (CHIP_EN)
- new net ESP32_LNA_IN: U11.1 (LNA_IN)
- new net ESP32_MISO: U11.9 (MTMS)
- new net ESP32_MOSI: U11.8 (GPIO3)
- new net ESP32_NSS: R16.2, U11.10 (MTDI)
- new net ESP32_SCK: U11.6 (GPIO2)
- new net ESP32_USB_DN: R20.1, U1.7 (DN2)
- new net ESP32_USB_DP: R18.1, U1.3 (DP2)
- new net ESP32_VDD: C48.1, U11.18 (VDD_SPI)
- new net ESP32_XTAL_N: C18.2, U11.29 (XTAL_N), X2.3 (OSC2)
- new net ESP32_XTAL_P: C22.1, U11.30 (XTAL_P), X2.1 (OSC1)
- new net RF_VDD: C42.1, C43.1, C44.1, C47.1, C51.1, C52.1, C53.1, R16.1, U11.11 (VDD3P3_RTC), U11.17 (VDD3P3_CPU), U11.2 (VDD3P3), U11.3 (VDD3P3), U11.31 (VDDA), U11.32 (VDDA), U13.5 (OUT)
- new net STM32_INA_ALERT: U2.3 (Alert)
- new net STM32_ISP2_MISO: J6.5 (Pin_5)
- new net STM32_TIM2_CH2: J5.4 (Pin_4)
- new net STM32_USB_DN: R17.1, U1.8 (DN1)
- new net STM32_USB_DP: R19.1, U1.2 (DP1)
- new net SX_DIO0: U11.13 (MTDO)
- new net SX_DIO1: R21.2, U11.14 (GPIO8)
- new net SX_RESET: U11.12 (MTCK)
- new net TP3U_SEL: J1.2 (Pin_2), R7.2, U1.1 (SEL)
- new net USB_CC1: U6.7 (CC1), USB1.A5 (CC1)
- new net USB_CC2: U6.6 (CC2), USB1.B5 (CC2)
- new net USB_DN: U1.6 (DN), U6.5 (DM), USB1.A7 (DN1), USB1.B7 (DN2)
- new net USB_DP: U1.4 (DP), U6.4 (DP), USB1.A6 (DP1), USB1.B6 (DP2)
- no-connect marks 0 -> 13
Other:
- note added: "5V Buck Converter"
- note added: "BMP388"
- note added: "Battery Protection"
- note added: "Connectors"
- note added: "ESP32 BOOT & EN"
- note added: "ESP32 Crystal"
- note added: "IMU ICM-42605"
- note added: "Low Drop Out Regulator"
- note added: "STM32 Crystal"
- note added: "STM32 Current Sense"
- note added: "STM32 ESP32 USB and Switching"
- note added: "STM32 LED"
- note added: "STM32 Reset & Boot"
- note added: "STM32 Serial NoR Flash"
- note added: "USB PD"
- note added: "USB Power OR-ing"
- moved on the sheet: L1, U12, U3

Commit message: feat: ESP32-C3 Antenna
Parts:
- removed C1, C23, C43, C44, C47, C48, C5, C52, C7, C8, C9: 100nF, Capacitor_SMD:C_0603_1608Metric, symbol Device:C_Small
- removed C10, C45: 2.2uF, Capacitor_SMD:C_0603_1608Metric, symbol Device:C_Small
- removed C11, C12: 22uF, Capacitor_SMD:C_0805_2012Metric, symbol Device:C_Small
- removed C13: 4.7uF, Capacitor_SMD:C_0603_1608Metric, symbol Device:C_Small
- removed C15, C19, C20: 10uF, Capacitor_SMD:C_0805_2012Metric, symbol Device:C_Small
- removed C17: 1uF, Capacitor_SMD:C_0603_1608Metric, symbol Device:C_Small
- removed C18, C22: 22pF, Capacitor_SMD:C_0603_1608Metric, symbol Device:C_Small
- removed C2, C3, C4: 100uF, Capacitor_SMD:C_1206_3216Metric, symbol Device:C_Small
- removed C42, C51: 10nF, Capacitor_SMD:C_0603_1608Metric, symbol Device:C_Small
- removed C53, C54: 10uF, Capacitor_SMD:C_0603_1608Metric, symbol Device:C_Small
- removed C55, C56: 22uF, Capacitor_SMD:C_0603_1608Metric, symbol Device:C_Small
- removed C6: 200pF, Capacitor_SMD:C_0603_1608Metric, symbol Device:C_Small
- removed D1: XL-1608PGC-06, easyeda2kicad:LED0603-RD_GREEN, symbol easyeda2kicad:XL-1608PGC-06
- removed FB3: FerriteBead, Inductor_SMD:L_0603_1608Metric, symbol Device:FerriteBead_Small
- removed J1: Jumper Pin Select, easyeda2kicad:PinHeader_1x03_P2.54mm_Vertical_Custom, symbol Connector:Conn_01x03_Pin
- removed L1: MHCI06030-1R5M-R8A, easyeda2kicad:IND-SMD_L7.3-W6.6, symbol easyeda2kicad:MHCI06030-1R5M-R8A
- removed Q1, Q2: AO3011A, easyeda2kicad:SOT-23-3_L2.9-W1.6-P1.90-LS2.8-BR, symbol easyeda2kicad:AO3011A
- removed R1: 100K, symbol Device:R_Small
- removed R11, R13, R16, R21, R7: 10K, Resistor_SMD:R_0603_1608Metric, symbol Device:R_Small
- removed R14, R22: 100, Resistor_SMD:R_0603_1608Metric, symbol Device:R_Small
- removed R18, R20: 22, Resistor_SMD:R_0603_1608Metric, symbol Device:R_Small
- removed R2: LR2512D-0.5MR, easyeda2kicad:RES-SMD_L6.4-W3.2_C500733, symbol easyeda2kicad:LR2512D-3W-0.5MR-1%
- removed R3, R5: 10K, symbol Device:R_Small
- removed R4: 1K, symbol Device:R_Small
- removed R6: 12K, symbol Device:R_Small
- removed R8: 1K, Resistor_SMD:R_0603_1608Metric, symbol Device:R_Small
- removed SW3, SW4: TACTILE SWITCH, easyeda2kicad:KEY-SMD_L4.0-W3.0-LS4.9-1, symbol easyeda2kicad:HX3X4X2-2P-1.6NTACTILESWITCH
- removed U1: TP3USB30M10, easyeda2kicad:MSOP-10_L3.0-W3.0-P0.50-LS4.9-BL, symbol easyeda2kicad:TP3USB30M10
- removed U11: ESP32-C3FH4, easyeda2kicad:QFN-32_L5.0-W5.0-P0.50-TL-EP3.7, symbol easyeda2kicad:ESP32-C3FH4
- removed U13: TLV75733PDBVR, easyeda2kicad:SOT-23-5_L2.9-W1.6-P0.95-LS2.8-BL, symbol easyeda2kicad:TLV75733PDBVR
- removed U2: INA226AIDGSR, easyeda2kicad:MSOP-10_L3.0-W3.0-P0.50-LS5.0-BL, symbol easyeda2kicad:INA226AIDGSR
- removed U3: SY8368AQQC, easyeda2kicad:QFN-12_L3.0-W3.0-P0.45-TL-EP, symbol easyeda2kicad:SY8368AQQC
- removed U4, U9: MX74610T, easyeda2kicad:SOT-23-6_L2.9-W1.6-P0.95-LS2.8-BL-1, symbol easyeda2kicad:MX74610T
- removed U5: SP1117, Package_TO_SOT_SMD:SOT-223-3_TabPin2, symbol Regulator_Linear:AMS1117
- removed U6: CH224K, Package_SO:SSOP-10-1EP_3.9x4.9mm_P1mm_EP2.1x3.3mm, symbol Interface_USB:CH224K
- removed USB1: USB-TYPE-C-018, easyeda2kicad:USB-C_SMD-TYPE-C-31-M-12, symbol easyeda2kicad:USB-TYPE-C-018
- removed X2: X322540MPB4SI, easyeda2kicad:OSC-SMD_4P-L3.2-W2.5-BL_SIT8008BI, symbol easyeda2kicad:X322540MPB4SI
- added R9: 100, Resistor_SMD:R_0603_1608Metric, symbol Device:R_Small
- renumbered C46 to C1, C24 to C10, C41 to C11, C28 to C12, C33 to C13, C25 to C14, C29 to C15, C34 to C16, C37 to C17, C30 to C18, C35 to C19, C21 to C2, C38 to C20, C31 to C21, C36 to C22, C39 to C23, C27 to C24, C26 to C25, C32 to C26, C16 to C3, C49 to C4, C50 to C5, C14 to C6, C40 to C7, C57 to C8, C58 to C9, D3 to D1, FB2 to FB1, FB1 to FB2, J5 to J1, J8 to J2, J7 to J4, J4 to J5, J2 to J6, J6 to J7, Q3 to Q1, R25 to R1, R12 to R10, R10 to R2, R15 to R3, R9 to R4, R17 to R5, R19 to R6, R23 to R7, R24 to R8, SW2 to SW1, SW1 to SW2, U10 to U1, U12 to U2, U7 to U3, U8 to U4
Connections:
- net STM32_TIM2_CH2 is gone; now on net STM32_TIM1_CH2: J1.4 (Pin_4)
- net at D2.2 (A): now also R9.2
- net STM32_LED: no longer names the net of U2.7 (PC13)
- net STM32_LED: now also R9.1
- no-connect marks 13 -> 0
Other:
- added sheet PowerSupply (CodeName02_PowerSupply.kicad_sch)
- added sheet RF Microcontroller (CodeName02_RF.kicad_sch)
- added sheet USB (CodeName02_USB.kicad_sch)
- note removed: "5V Buck Converter"
- note removed: "Battery Protection"
- note removed: "ESP32 BOOT & EN"
- note removed: "ESP32 Crystal"
- note removed: "Low Drop Out Regulator"
- note removed: "STM32 Current Sense"
- note removed: "STM32 ESP32 USB and Switching"
- note removed: "STM32 LED"
- note removed: "USB PD"
- note removed: "USB Power OR-ing"
- moved on the sheet: C1, C10, C11, C12, C13, C14, C15, C16, C17, C18, C19, C2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

Commit message: feat: finalize
Parts:
- removed U3: XT25F128FWOIGT-W, easyeda2kicad:WSON-8_L6.0-W5.0-P1.27-BL-EP, symbol easyeda2kicad:XT25F128FWOIGT-W
- added J10: AUX Timer Connection, easyeda2kicad:PinHeader_3Row_Custom, symbol Connector:Conn_01x18_Pin
- added U3: W25Q128JVPIQTR, easyeda2kicad:WSON-8_L6.0-W5.0-P1.27-BL, symbol easyeda2kicad:W25Q128JVPIQTR
- J2: footprint Connector_JST:JST_GH_SM04B-GHS-TB_1x04-1MP_P1.25mm_Horizontal -> Connector_JST:JST_GH_BM04B-GHS-TBT_1x04-1MP_P1.25mm_Vertical
Connections:
- net +3.3V: now also U3.8 (VCC)
- net +5V: now also J10.11 (Pin_11), J10.14 (Pin_14), J10.17 (Pin_17), J10.2 (Pin_2), J10.5 (Pin_5), J10.8 (Pin_8)
- net GND: now also J10.12 (Pin_12), J10.15 (Pin_15), J10.18 (Pin_18), J10.3 (Pin_3), J10.6 (Pin_6), J10.9 (Pin_9), U3.4 (GND), U3.9 (EP)
- net STM32_ISP2_MISO: now also U2.53 (PB14)
- net STM32_QSPI_CLK: now also U3.6 (CLK)
- net STM32_QSPI_IO0: now also U3.5 (DI/IO0)
- net STM32_QSPI_IO1: now also U3.2 (DO/IO1)
- net STM32_QSPI_IO2: now also U3.3 (#WP/IO2)
- net STM32_QSPI_IO3: now also U3.7 (#HOLD-OR-#REST/IO3)
- net STM32_QSPI_NCS: now also U3.1 (#CS)
- net STM32_TIM4_CH1: now also J10.13 (Pin_13)
- net STM32_TIM4_CH2: now also J10.16 (Pin_16)
- net STM32_TIM5_CH1: now also J10.1 (Pin_1)
- net STM32_TIM5_CH2: now also J10.4 (Pin_4)
- net STM32_TIM5_CH3: now also J10.7 (Pin_7)
- net STM32_TIM5_CH4: now also J10.10 (Pin_10)
- net STM32_INA_ALERT: now reaches U2.47 (PB11)
- net STM32_SDMMC1_CK renamed STM32_SDMMC1_CLK
Other:
- moved on the sheet: C24, D2, R10, R9
