File: CodeName02_PowerSupply.kicad_sch (KiCad schematic)
At the start: 26 parts, among them Q2 AO3011A, U5 SP1117, U6 MX74610T, U7 INA226AIDGSR, U8 SY8368AQQC

Commit message: feat: finalize
Parts:
- added TP1: TestPoint VBAT_RAW, TestPoint:TestPoint_Pad_D2.0mm, symbol Connector:TestPoint
- added TP2: TestPoint SYS_POWER, TestPoint:TestPoint_Pad_D2.0mm, symbol Connector:TestPoint
- added TP3: TestPoint 5V, TestPoint:TestPoint_Pad_D2.0mm, symbol Connector:TestPoint
- added TP4: TestPoint 3.3V, TestPoint:TestPoint_Pad_D2.0mm, symbol Connector:TestPoint
Connections:
- net +3.3V: now also TP4.1
- net +5V: now also TP3.1
- net +BATT_RAW: now also TP1.1
- net +SYS_POWER: now also TP2.1
Other:
- note added: "Test Point Power"
