File: CodeName02_RF.kicad_sch (KiCad schematic)
At the start: 32 parts, among them SW3 TACTILE SWITCH, SW4 TACTILE SWITCH, U12 ESP32-C3FH4, U13 TLV75733PDBVR, X2 X322540MPB4SI

Commit message: feat: finalize
Parts:
- added C61, C62, C66, C68: 10nF, Capacitor_SMD:C_0603_1608Metric, symbol Device:C_Small
- added C63, C65: 100nF, Capacitor_SMD:C_0603_1608Metric, symbol Device:C_Small
- added C64: 470nF, Capacitor_SMD:C_0603_1608Metric, symbol Device:C_Small
- added C67: 47pF, Capacitor_SMD:C_0402_1005Metric, symbol Device:C_Small
- added FL1: 2450FM07D0034T, easyeda2kicad:FILTER-SMD_4P-L1.0-W0.5-L, symbol easyeda2kicad:2450FM07D0034T
- added J9: Conn_Coaxial_Small, Connector_Coaxial:U.FL_Hirose_U.FL-R-SMT-1_Vertical, symbol Connector:Conn_Coaxial_Small
- added U14: SX1280IMLTRT, easyeda2kicad:QFN-24_L4.0-W4.0-P0.50-BL-EP2.6, symbol easyeda2kicad:SX1280IMLTRT
- added X3: XC21M4-52.000-F10NNHPL, easyeda2kicad:CRYSTAL-SMD_4P-L2.0-W1.6-BL, symbol easyeda2kicad:XC21M4-52.000-F10NNHPL
- L2: footprint LED_SMD:LED_0402_1005Metric -> Inductor_SMD:L_0402_1005Metric
Connections:
- net ESP32_MISO: now also U14.16 (MISO_TX)
- net ESP32_MOSI: now also U14.17 (MOSI_RX)
- net ESP32_NSS: now also U14.19 (NSS_CTS)
- net ESP32_SCK: now also U14.18 (SCK_RTSN)
- net GND: now also C61.2, C62.2, C63.2, C64.2, C65.2, C66.2, C67.2, C68.2, FL1.2 (GND), FL1.4 (GND), J9.2 (Ext), U14.13 (GND), U14.20 (GND), U14.21 (GND), U14.23 (GND), U14.24 (GND), U14.25 (GND), U14.5 (GND), X3.2 (GND), X3.4 (GND)
- net RF_VDD: now also C63.1, C65.1, C66.1, C67.1, C68.1, U14.11 (VBAT_IO), U14.15 (VBAT)
- net SX_DIO1: now also U14.8 (DIO1)
- net SX_RESET: now also U14.3 (NRESET)
- net SX_DIO0 renamed SX_BUSY
- net SX_BUSY: now also U14.7 (BUSY)
- new net: C61.1, U14.1 (VR_PA)
- new net: C62.1, C64.1, U14.12 (DCC_FB), U14.2 (VDD_IN)
- new net: FL1.1 (IN), U14.22 (RFIO)
- new net: FL1.3 (OUT), J9.1 (In)
- new net SX_XTA: U14.4 (XTA), X3.1
- new net SX_XTB: U14.6 (XTB), X3.3
- no-connect marks 9 -> 12
Other:
- note added: "SX1280 Crystal"
- moved on the sheet: AE1, C45, C47, C48, C51, C52, C53, C54, C55, C59, C60, D3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
